File: output.kicad_sch (KiCad schematic)
At the start: 8 parts, among them J6 Screw_Terminal_01x02, K1 Relay_SPST-NO, Q1 Q_NPN_BCE

Commit message: Schematic ready; PCB needs silkscreen
Parts:
- D7, D8: footprint (none) -> Diode_THT:D_DO-41_SOD81_P2.54mm_Vertical_AnodeUp
- D9: footprint (none) -> LED_THT:LED_D3.0mm
- J7: renamed from J6; footprint (none) -> TerminalBlock_RND:TerminalBlock_RND_205-00001_1x02_P5.00mm_Horizontal
- K1: footprint (none) -> Relay_THT:Relay_SPST_SANYOU_SRD_Series_Form_A
- Q1: value Q_NPN_BCE -> Q_NPN_EBC; footprint (none) -> Package_TO_SOT_THT:TO-92; symbol Device:Q_NPN_BCE -> Device:Q_NPN_EBC
- R8, R9: footprint (none) -> Resistor_THT:R_Axial_DIN0204_L3.6mm_D1.6mm_P1.90mm_Vertical
Connections:
- net GND: now also Q1.1 (E); no longer Q1.3 (E)
- net at D8.1 (K), K1.A2, R8.2: now also Q1.3 (C); no longer Q1.2 (C)
- net at R9.2: now also Q1.2 (B); no longer Q1.1 (B)
Changed lines of the file:
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@@
 			)
 		)
-		(property "Footprint" ""
+		(property "Footprint" "Diode_THT:D_DO-41_SOD81_P2.54mm_Vertical_AnodeUp"
 			(at 153.67 99.06 0)
 			(effects
@@
 			)
 		)
-		(property "Footprint" ""
+		(property "Footprint" "Diode_THT:D_DO-41_SOD81_P2.54mm_Vertical_AnodeUp"
 			(at 153.67 91.44 0)
 			(effects
@@
 			)
 		)
-		(property "Footprint" ""
+		(property "Footprint" "Resistor_THT:R_Axial_DIN0204_L3.6mm_D1.6mm_P1.90mm_Vertical"
 			(at 165.1 109.728 90)
 			(effects
@@
 	)
 	(symbol
-		(lib_id "Device:Q_NPN_BCE")
+		(lib_id "Device:Q_NPN_EBC")
 		(at 156.21 107.95 0)
 		(mirror y)
@@
 			)
 		)
-		(property "Value" "Q_NPN_BCE"
+		(property "Value" "Q_NPN_EBC"
 			(at 151.13 109.2199 0)
 			(effects
@@
 			)
 		)
-		(property "Footprint" ""
+		(property "Footprint" "Package_TO_SOT_THT:TO-92"
 			(at 151.13 105.41 0)
 			(effects
@@
 			)
 		)
-		(property "Description" "NPN transistor, base/collector/emitter"
+		(property "Description" "NPN transistor, emitter/base/collector"
 			(at 156.21 107.95 0)
 			(effects
@@
 			)
 		)
-		(property "Footprint" ""
+		(property "Footprint" "LED_THT:LED_D3.0mm"
 			(at 162.56 91.44 0)
 			(effects
@@
 		(on_board yes)
 		(dnp no)
-		(property "Reference" "J6"
+		(property "Reference" "J7"
 			(at 116.586 90.678 0)
 			(effects
@@
 			)
 		)
-		(property "Footprint" ""
+		(property "Footprint" "TerminalBlock_RND:TerminalBlock_RND_205-00001_1x02_P5.00mm_Horizontal"
 			(at 116.84 96.52 0)
 			(effects
@@
 			(project "SolderTestPCB"
 				(path "/3f231ef2-6b13-4d44-9a8c-c6a44054681e/525a9041-6d36-487d-93ef-76e2dea8509b"
-					(reference "J6")
-					(unit 1)
-				)
-				(path "/3f231ef2-6b13-4d44-9a8c-c6a44054681e/766f1a07-b6c9-4dfc-af2a-10aff4e96ec5"
-					(reference "J8")
+					(reference "J7")
+					(unit 1)
+				)
+				(path "/3f231ef2-6b13-4d44-9a8c-c6a44054681e/766f1a07-b6c9-4dfc-af2a-10aff4e96ec5"
+					(reference "J9")
 					(unit 1)
 				)
@@
 			)
 		)
-		(property "Footprint" ""
+		(property "Footprint" "Resistor_THT:R_Axial_DIN0204_L3.6mm_D1.6mm_P1.90mm_Vertical"
 			(at 164.338 99.06 90)
 			(effects
@@
 			)
 		)
-		(property "Footprint" ""
+		(property "Footprint" "Relay_THT:Relay_SPST_SANYOU_SRD_Series_Form_A"
 			(at 128.27 96.52 0)
 			(effects

Commit message: PCB Layout finished (RTM)
Parts:
- D7, D8: footprint Diode_THT:D_DO-41_SOD81_P2.54mm_Vertical_AnodeUp -> Diode_THT:D_DO-15_P10.16mm_Horizontal
Changed lines of the file:
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@@
 			)
 		)
-		(property "Footprint" "Diode_THT:D_DO-41_SOD81_P2.54mm_Vertical_AnodeUp"
+		(property "Footprint" "Diode_THT:D_DO-15_P10.16mm_Horizontal"
 			(at 153.67 99.06 0)
 			(effects
@@
 			)
 		)
-		(property "Footprint" "Diode_THT:D_DO-41_SOD81_P2.54mm_Vertical_AnodeUp"
+		(property "Footprint" "Diode_THT:D_DO-15_P10.16mm_Horizontal"
 			(at 153.67 91.44 0)
 			(effects
